File: KiCAD/Ceinture Respiration/MCU.kicad_sch (KiCad schematic)
At the start: 0 parts

Commit message: First draft PCB and sch
Parts:
- added A1: Arduino_Nano_v3.x, Module:Arduino_Nano, symbol MCU_Module:Arduino_Nano_v3.x
Connections:
- new net +9V: A1.30 (VIN)
- new net GND: A1.29 (GND), A1.4 (GND)
Changed lines of the file:
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@@
-(kicad_sch (version 20211123) (generator eeschema)
+(kicad_sch (version 20230121) (generator eeschema)
   (paper "A4")
+  (junction (at 138.43 118.11) (diameter 0) (color 0 0 0 0)
+  )
+  (wire (pts (xy 138.43 113.03) (xy 138.43 118.11))
+    (stroke (width 0) (type default))
+  )
+  (wire (pts (xy 135.89 118.11) (xy 138.43 118.11))
+    (stroke (width 0) (type default))
+  )
+  (wire (pts (xy 133.35 55.88) (xy 133.35 62.23))
+    (stroke (width 0) (type default))
+  )
+  (wire (pts (xy 135.89 113.03) (xy 135.89 118.11))
+    (stroke (width 0) (type default))
+  )
+  (wire (pts (xy 138.43 118.11) (xy 138.43 121.92))
+    (stroke (width 0) (type default))
+  )
+  (symbol (lib_id "power:GND") (at 138.43 121.92 0) (unit 1)
+    (in_bom yes) (on_board yes) (dnp no) (fields_autoplaced)
+    (property "Reference" "#PWR02" (at 138.43 128.27 0)
+      (effects (font (size 1.27 1.27)) hide)
+    )
+    (property "Value" "GND" (at 138.43 127 0)
+      (effects (font (size 1.27 1.27)))
+    )
+    (property "Footprint" "" (at 138.43 121.92 0)
+      (effects (font (size 1.27 1.27)) hide)
+    )
+    (property "Datasheet" "" (at 138.43 121.92 0)
+      (effects (font (size 1.27 1.27)) hide)
+    )
+    (pin "1")
+    (instances
+      (project "Ceinture Respiration"
+        (path "/5bd6870d-598f-44db-8dd6-81ffc3a9b2d4/6e64942f-9b80-4043-a53a-e59ed80f674d"
+          (reference "#PWR02") (unit 1)
+        )
+      )
+    )
+  )
+  (symbol (lib_id "MCU_Module:Arduino_Nano_v3.x") (at 135.89 87.63 0) (unit 1)
+    (in_bom yes) (on_board yes) (dnp no) (fields_autoplaced)
+    (property "Reference" "A1" (at 140.3859 113.03 0)
+      (effects (font (size 1.27 1.27)) (justify left))
+    )
+    (property "Value" "Arduino_Nano_v3.x" (at 140.3859 115.57 0)
+      (effects (font (size 1.27 1.27)) (justify left))
+    )
+    (property "Footprint" "Module:Arduino_Nano" (at 135.89 87.63 0)
+      (effects (font (size 1.27 1.27) italic) hide)
+    )
+    (property "Datasheet" "http://www.mouser.com/pdfdocs/Gravitech_Arduino_Nano3_0.pdf" (at 135.89 87.63 0)
+      (effects (font (size 1.27 1.27)) hide)
+    )
+    (pin "1")
+    (pin "10")
+    (pin "11")
+    (pin "12")
+    (pin "13")
+    (pin "14")
+    (pin "15")
+    (pin "16")
+    (pin "17")
+    (pin "18")
+    (pin "19")
+    (pin "2")
+    (pin "20")
+    (pin "21")
+    (pin "22")
+    (pin "23")
+    (pin "24")
+    (pin "25")
+    (pin "26")
+    (pin "27")
+    (pin "28")
+    (pin "29")
+    (pin "3")
+    (pin "30")
+    (pin "4")
+    (pin "5")
+    (pin "6")
+    (pin "7")
+    (pin "8")
+    (pin "9")
+    (instances
+      (project "Ceinture Respiration"
+        (path "/5bd6870d-598f-44db-8dd6-81ffc3a9b2d4/6e64942f-9b80-4043-a53a-e59ed80f674d"
+          (reference "A1") (unit 1)
+        )
+      )
+    )
+  )
+  (symbol (lib_id "power:+9V") (at 133.35 55.88 0) (unit 1)
+    (in_bom yes) (on_board yes) (dnp no) (fields_autoplaced)
+    (property "Reference" "#PWR01" (at 133.35 59.69 0)
+      (effects (font (size 1.27 1.27)) hide)
+    )
+    (property "Value" "+9V" (at 133.35 50.8 0)
+      (effects (font (size 1.27 1.27)))
+    )
+    (property "Footprint" "" (at 133.35 55.88 0)
+      (effects (font (size 1.27 1.27)) hide)
+    )
+    (property "Datasheet" "" (at 133.35 55.88 0)
+      (effects (font (size 1.27 1.27)) hide)
+    )
+    (pin "1")
+    (instances
+      (project "Ceinture Respiration"
+        (path "/5bd6870d-598f-44db-8dd6-81ffc3a9b2d4/6e64942f-9b80-4043-a53a-e59ed80f674d"
+          (reference "#PWR01") (unit 1)
+        )
+      )
+    )
+  )
 )
