File: KiCAD/Ceinture Respiration/PSU.kicad_sch (KiCad schematic)
At the start: 1 part

Commit message: First draft PCB and sch
Parts:
- added BT1: BH9VPC, BAT_BH9VPC, symbol CeintureRespAT:BH9VPC
- added PS1: RS3-0505D, CONV_RS3-0505D, symbol CeintureRespAT:RS3-0505D
Connections:
- net +BATT: now reaches SW?.1 (A)
- net +BATT: now also PS1.2 (+VIN)
- net at SW?.2 (B): now also BT1.+
- new net +5VA: PS1.6 (+VOUT)
- new net -5V: PS1.8 (-VOUT)
- new net GND: PS1.7 (COM)
- new net GND2: BT1.-, PS1.1 (-VIN), PS1.3 (CTRL)
Other:
- note added: "RS3-0505D avec une batterie 9V"
- note removed: "Gestion Li-Po"
- note removed: "Power supply du capteur, on doit connaitre la consomation courant -TPS65131RGET pour +/-12v, on aura autour de 250mA -Sinon PQDE6W-D"
- note removed: "Références https://download.mikroe.com/documents/add-on-boards/click/boost-inv-2/boost-inv-2-click-schematic-v100.pdf"
- moved on the sheet: SW?
