File: KiCAD/Ceinture Respiration/Ceinture Respiration.kicad_sch (KiCad schematic)
At the start: 5 parts, among them J1 Conn_01x10_Pin, J2 Conn_01x10_Socket

Commit message: PCB sent for production
See latest production files.
Parts:
- F1, F2, F3: LCSC (none) -> C2844464
Changed lines of the file:
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@@
+      (effects (font (size 1.27 1.27)) hide)
+    )
+    (property "LCSC" "C2844464" (at 137.16 118.745 0)
       (effects (font (size 1.27 1.27)) hide)
     )
@@
     )
     (property "Datasheet" "~" (at 135.89 97.155 0)
+      (effects (font (size 1.27 1.27)) hide)
+    )
+    (property "LCSC" "C2844464" (at 135.89 97.155 90)
       (effects (font (size 1.27 1.27)) hide)
     )
@@
       (effects (font (size 1.27 1.27)) hide)
     )
+    (property "LCSC" "C2844464" (at 137.16 114.935 0)
+      (effects (font (size 1.27 1.27)) hide)
+    )
