File: KiCAD/Main board/Ceinture_respiration_Main/Ceinture_respiration_Main.kicad_sch (KiCad schematic)
At the start: 4 parts, among them J2 Conn_01x10_Socket

Commit message: modifié info Part number du main board pour faciliter la génération de BOM non JLC
Parts:
- J2: LCSC (none) -> C2897373
Changed lines of the file:
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@@
+			)
+		)
+		(property "LCSC" "C2897373"
+			(at 132.715 92.075 0)
+			(effects
+				(font
+					(size 1.27 1.27)
+				)
+				(hide yes)
 			)
 		)
