File: KiCAD/Main board/Ceinture_respiration_Main/MCU.kicad_sch (KiCad schematic)
At the start: 8 parts, among them J3 Conn_01x06_Pin, J4 Conn_01x06_Pin, J5 Conn_01x06_Pin

Commit message: modifié info Part number du main board pour faciliter la génération de BOM non JLC
Parts:
- J3, J4, J5: MPN (none) -> Grove Conn
Changed lines of the file:
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@@
+			)
+		)
+		(property "MPN" "Grove Conn"
+			(at 222.885 105.41 0)
+			(effects
+				(font
+					(size 1.27 1.27)
+				)
+				(hide yes)
 			)
 		)
@@
 			)
 		)
+		(property "MPN" "Grove Conn"
+			(at 222.885 128.905 0)
+			(effects
+				(font
+					(size 1.27 1.27)
+				)
+				(hide yes)
+			)
+		)
 		(pin "1"
 		)
@@
 			)
 		)
+		(property "MPN" "Grove Conn"
+			(at 222.885 79.375 0)
+			(effects
+				(font
+					(size 1.27 1.27)
+				)
+				(hide yes)
+			)
+		)
