File: KiCAD/Shield/Ceinture_respiration_Shield/SHIELD_RESPIRATION.kicad_sch (KiCad schematic)
At the start: 3 parts, among them J6 DIN-8, J7 DIN-8

Commit message: Changé # pièce switch sur main board poru utiliser pièces en stock.
Parts:
- J6, J7: MPN (none) -> SDS-80J
- PS1: Field11 (none) -> MPN
Changed lines of the file:
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@@
+			)
+		)
+		(property "MPN" "SDS-80J"
+			(at 42.545 53.975 0)
+			(effects
+				(font
+					(size 1.27 1.27)
+				)
+				(hide yes)
 			)
 		)
@@
 			)
 		)
+		(property "MPN" "SDS-80J"
+			(at 81.28 53.975 0)
+			(effects
+				(font
+					(size 1.27 1.27)
+				)
+				(hide yes)
+			)
+		)
 		(pin "1"
 		)
@@
 			(at 135.255 53.975 0)
 			(effects
+				(font
+					(size 1.27 1.27)
+				)
+				(hide yes)
+			)
+		)
+		(property "Field11" "MPN"
+			(at 135.255 53.975 0)
+			(effects
