File: KiCAD/Shield/Ceinture_respiration_Shield/Ceinture_respiration_Shield.kicad_sch (KiCad schematic)
At the start: 1 part, among them J1 Conn_01x10_Pin

Commit message: ajouté fichiers oublier
Parts:
- J1: MPN (none) -> 2011-1X10G00SB
Changed lines of the file:
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@@
+			)
+		)
+		(property "MPN" "2011-1X10G00SB"
+			(at 163.83 79.375 0)
+			(effects
+				(font
+					(size 1.27 1.27)
+				)
+				(hide yes)
 			)
 		)
